File: PCB/v2.6/WeatherChimesV2.6.brd (EAGLE design)
At the start: 102.8 x 78.9 mm, 24 parts, among them U1 MS5803-02BA

Commit message: Add files via upload
Parts:
- removed JP1: (no value), microbuilder:1X11_ROUND_76
- removed U$13, U$14, U$15, U$16: MOUNTINGHOLE2.5, microbuilder:MOUNTINGHOLE_2.5_PLATED
- added BATT: JST 2PH, adafruit:JST-PH-2-SMT-RA
- added C5, C6: 10uF, adafruit:C0805K
- added D2: SK34A, microbuilder:SMADIODE
- added JP8: (no value), pinhead:1X02
- added R11, R4, R7, R8: 10K, adafruit:M0805
- added R3, R9: 1K, adafruit:M0805
- added X4: BQ24074, adafruit_power:QFN16_3MM
- moved U$1 1.27 mm to (63.5, 59.7)
- moved J1 0.76 mm to (2.03, 52.1)
- moved J2 0.76 mm to (2.03, 41.9)
- moved J3 0.76 mm to (2.03, 31.8)
- moved J4 0.76 mm to (2.03, 21.6)
- moved SW_D11 0.76 mm to (3.30, 61.0)
Connections:
- new net !CE: R8.1, X4.4
- new net !CHG: R7.1, X4.9
- new net !PGOOD: R11.1, X4.7
- new net CHARGER_IN: D2.A
- new net ILIM: R3.1, X4.12
- new net ISET: R9.1, X4.16
- new net ITERM: R4.1, X4.15
- new net N$1: X4.5
- new net N$2: D2.C, X4.13
- new net THERM: JP8.1, X4.1
- new net VLIPO: BATT.1, X4.2, X4.3
- net GND: now also BATT.2, JP8.2, R3.2, R4.2, R8.2, R9.2, X4.14, X4.6, X4.8, X4.THERMAL; no longer JP1.1, JP1.10, JP1.3
- net PGOOD: no longer JP1.6
- net VBAT: now also X4.10, X4.11; no longer JP1.4
Routing:
- net PGOOD: track 62.3 -> 0.00 mm
- net SCL: track 184.2 -> 141.3 mm, vias 0 -> 2
- net SDA: track 157.0 -> 183.8 mm, vias 0 -> 2
- net !PGOOD: track 0.00 -> 13.7 mm
- net RX: track 73.5 -> 62.2 mm
- net THERM: track 0.00 -> 10.4 mm
- net !CE: track 0.00 -> 10.2 mm, vias 0 -> 2
- net N$2: track 0.00 -> 10.1 mm
- net !CHG: track 0.00 -> 9.76 mm
- net VLIPO: track 0.00 -> 7.72 mm
- net VBAT: track 102.0 -> 109.2 mm, vias 0 -> 2
- net ITERM: track 0.00 -> 4.78 mm
- net ILIM: track 0.00 -> 3.44 mm
- net ISET: track 0.00 -> 2.63 mm
- net VCC: track 177.9 -> 180.2 mm
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Other:
- board text added: "I2C"
- board text added: "SDI"
- board text added: "SOLAR CHARGER"
- board text added: "Winnie Woo"
- board text removed: "CE"
- board text removed: "CHG"
- board text removed: "ISET"
- board text removed: "LIPO"
- board text removed: "OUT"
- board text removed: "PGOOD"
- board text removed: "SDI12_A0"
- board text removed: "SOLAR CHARGER this side"
- board text removed: "THERM"
- board text removed: "VBUS"
- board text removed: "Woo, Udell 2022"

Commit message: Add files via upload
Parts:
- moved HP1 3.81 mm to (71.1, 62.2)
- moved HP2 3.81 mm to (91.4, 52.1)
- moved U$4 0.80 mm to (97.0, 75.9)
- moved U$5 0.80 mm to (97.0, 4.83)
Routing:
- net SDA: track 183.8 -> 174.1 mm
- net VCC: track 180.2 -> 176.4 mm
- net VBAT: track 109.2 -> 105.4 mm
- net SDI: track 75.9 -> 72.1 mm
- net SCL: track 141.3 -> 137.4 mm
- net RX: track 62.2 -> 58.4 mm
- net 4GONOFF: track 66.2 -> 62.3 mm
- net TX: track 66.4 -> 62.6 mm
- net 5VRAIL: track 49.1 -> 48.2 mm
Other:
- board size 102.8 x 78.9 mm -> 101.8 x 79 mm

Commit message: Add files via upload
Parts:
- moved U$5 2.16 mm to (94.9, 4.95)
- moved U$4 2.16 mm to (94.9, 76.1)
- moved HP1 1.52 mm to (69.6, 62.2)
- moved HP2 1.52 mm to (89.9, 52.1)
Routing:
- net SDA: track 174.1 -> 169.5 mm
- net VCC: track 176.4 -> 174.2 mm
- net TX: track 62.6 -> 61.0 mm
- net SDI: track 72.1 -> 70.6 mm
- net SCL: track 137.4 -> 135.9 mm
- net 5VRAIL: track 48.2 -> 46.8 mm
- net VBAT: track 105.4 -> 104.3 mm
- net RX: track 58.4 -> 57.4 mm
Other:
- board size 101.8 x 79 mm -> 99.3 x 79 mm

Commit message: Add files via upload
Routing:
- net SCL: track 135.9 -> 137.3 mm
- net RX: track 57.4 -> 58.7 mm
- net 5VRAIL: track 46.8 -> 47.5 mm
Changed lines of the file:
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@@
 <contactref element="HP1" pad="14"/>
 <wire x1="62.19270625" y1="23.749" x2="15.621" y2="23.749" width="0.2032" layer="1"/>
-<wire x1="63.00550625" y1="22.9362" x2="62.19270625" y2="23.749" width="0.2032" layer="1"/>
-<wire x1="64.10206875" y1="22.9362" x2="63.00550625" y2="22.9362" width="0.2032" layer="1"/>
-<wire x1="64.10206875" y1="22.9362" x2="69.596" y2="28.43013125" width="0.2032" layer="1"/>
-<wire x1="69.596" y1="28.43013125" x2="69.596" y2="29.21" width="0.2032" layer="1"/>
+<wire x1="62.19270625" y1="23.749" x2="63.13250625" y2="22.8092" width="0.2032" layer="1"/>
+<wire x1="69.596" y1="29.21" x2="67.15006875" y2="26.76406875" width="0.2032" layer="1"/>
+<wire x1="65.9892" y1="22.8092" x2="67.15006875" y2="23.97006875" width="0.2032" layer="1"/>
+<wire x1="67.15006875" y1="23.97006875" x2="67.15006875" y2="26.76406875" width="0.2032" layer="1"/>
+<wire x1="63.13250625" y1="22.8092" x2="65.9892" y2="22.8092" width="0.2032" layer="1"/>
 <wire x1="15.621" y1="23.749" x2="15.24" y2="24.13" width="0" layer="19" extent="1-1"/>
 </signal>
@@
 <wire x1="69.08046875" y1="30.4546" x2="70.11153125" y2="30.4546" width="0.2032" layer="1"/>
 <wire x1="70.11153125" y1="30.4546" x2="70.8406" y2="29.72553125" width="0.2032" layer="1"/>
-<wire x1="70.8406" y1="29.72553125" x2="70.8406" y2="28.69446875" width="0.2032" layer="1"/>
+<wire x1="70.8406" y1="29.72553125" x2="70.8406" y2="27.94" width="0.2032" layer="1"/>
 <wire x1="15.24" y1="26.67" x2="61.81170625" y2="26.67" width="0.2032" layer="1"/>
 <wire x1="61.81170625" y1="26.67" x2="63.00550625" y2="27.8638" width="0.2032" layer="1"/>
-<wire x1="70.8406" y1="28.69446875" x2="69.596" y2="27.44986875" width="0.2032" layer="1"/>
-<wire x1="69.596" y1="27.44986875" x2="69.596" y2="26.67" width="0.2032" layer="1"/>
 <wire x1="63.00550625" y1="27.8638" x2="66.48966875" y2="27.8638" width="0.2032" layer="1"/>
 <wire x1="66.48966875" y1="27.8638" x2="69.08046875" y2="30.4546" width="0.2032" layer="1"/>
+<wire x1="70.8406" y1="27.94" x2="70.8406" y2="27.9146" width="0.2032" layer="1"/>
+<wire x1="70.8406" y1="27.9146" x2="69.596" y2="26.67" width="0.2032" layer="1"/>
 </signal>
 <signal name="SDA">
@@
 <wire x1="35.245" y1="53.655" x2="34.29" y2="53.655" width="0.2032" layer="1"/>
 <via x="65.786" y="38.1" extent="1-16" drill="0.508"/>
-<wire x1="89.916" y1="26.67" x2="78.97613125" y2="26.67" width="0.2032" layer="1"/>
+<wire x1="89.916" y1="26.67" x2="88.265" y2="25.019" width="0.2032" layer="1"/>
+<wire x1="88.265" y1="25.019" x2="80.62713125" y2="25.019" width="0.2032" layer="1"/>
 <wire x1="68.3514" y1="35.5346" x2="65.786" y2="38.1" width="0.2032" layer="1"/>
-<wire x1="78.97613125" y1="26.67" x2="70.11153125" y2="35.5346" width="0.2032" layer="1"/>
+<wire x1="80.62713125" y1="25.019" x2="70.11153125" y2="35.5346" width="0.2032" layer="1"/>
 <wire x1="70.11153125" y1="35.5346" x2="68.3514" y2="35.5346" width="0.2032" layer="1"/>
 <wire x1="65.786" y1="38.1" x2="64.262" y2="39.624" width="0.2032" layer="16"/>
@@
 <contactref element="U$1" pad="5V"/>
 <wire x1="89.916" y1="46.99" x2="72.136" y2="64.77" width="0.508" layer="1"/>
-<wire x1="72.136" y1="64.77" x2="67.31" y2="64.77" width="0.508" layer="1"/>
-<wire x1="67.31" y1="64.77" x2="67.31" y2="53.594" width="0.508" layer="1"/>
-<wire x1="67.31" y1="53.594" x2="63.5" y2="49.784" width="0.508" layer="1"/>
+<wire x1="66.04" y1="64.77" x2="72.136" y2="64.77" width="0.508" layer="1"/>
+<wire x1="63.5" y1="49.784" x2="66.04" y2="52.324" width="0.508" layer="1"/>
 <wire x1="63.5" y1="49.53" x2="63.5" y2="49.784" width="0.508" layer="1"/>
+<wire x1="66.04" y1="52.324" x2="66.04" y2="64.77" width="0.508" layer="1"/>
 </signal>
 <signal name="P13">
