File: PCB/v2.6/WeatherChimesV2.6.sch (EAGLE design)
At the start: 23 parts, among them U1 MS5803-02BA

Commit message: Add files via upload
Parts:
- removed U$6, U$7, U$8: MOUNTINGHOLE2.5, microbuilder:MOUNTINGHOLE2.5
Changed lines of the file:
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@@
 <part name="HP1" library="SparkFun-Connectors" library_urn="urn:adsk.eagle:library:513" deviceset="CONN_16" device="" package3d_urn="urn:adsk.eagle:package:38258/1"/>
 <part name="HP2" library="SparkFun-Connectors" library_urn="urn:adsk.eagle:library:513" deviceset="CONN_12" device="" package3d_urn="urn:adsk.eagle:package:38169/1"/>
-<part name="U$6" library="microbuilder" deviceset="MOUNTINGHOLE" device="2.5"/>
-<part name="U$7" library="microbuilder" deviceset="MOUNTINGHOLE" device="2.5"/>
 <part name="U1" library="PNNL_Probe" deviceset="MS5803-02BA" device=""/>
 <part name="JP5" library="pinhead_simple" deviceset="PINHD-1X1" device="" package3d_urn="urn:adsk.eagle:package:22485/2" value="GND"/>
@@
 <part name="SJ1" library="SparkFun-Jumpers" library_urn="urn:adsk.eagle:library:528" deviceset="JUMPER-SMT_3_1-NC_TRACE" device="_SILK" package3d_urn="urn:adsk.eagle:package:39288/1"/>
 <part name="SUPPLY8" library="supply2" library_urn="urn:adsk.eagle:library:372" deviceset="GND" device=""/>
-<part name="U$8" library="microbuilder" deviceset="MOUNTINGHOLE" device="2.5"/>
 </parts>
 <sheets>
@@
 <attribute name="NAME" x="203.2" y="55.372" size="1.778" layer="95" font="vector" rot="R180"/>
 </instance>
-<instance part="U$6" gate="G$1" x="160.02" y="-12.7" smashed="yes"/>
-<instance part="U$7" gate="G$1" x="167.64" y="-12.7" smashed="yes"/>
 <instance part="U1" gate="G$1" x="38.1" y="95.25" smashed="yes" grouprefs="MS580302BA">
 <attribute name="NAME" x="27.94" y="105.41" size="1.778" layer="95"/>
@@
 <attribute name="VALUE" x="60.325" y="98.425" size="1.778" layer="96"/>
 </instance>
-<instance part="U$8" gate="G$1" x="167.64" y="-17.78" smashed="yes"/>
 </instances>
 <busses>

Commit message: Add files via upload
Parts:
- removed JP1: (no value), microbuilder:HEADER-1X1176MIL
- added BATT: JST 2PH, adafruit:JST_2PIN-SMT-RA
- added C5, C6: 10uF, adafruit:C-USC0805K
- added D2: SK34A, microbuilder:DIODE-SCHOTTKYSMA
- added JP8: (no value), pinhead:PINHD-1X2
- added R11, R4, R7, R8: 10K, adafruit:R-US_M0805
- added R3, R9: 1K, adafruit:R-US_M0805
- added X4: BQ24074, adafruit_power:BQ24074
Connections:
- new net !CE: R8.1, X4.!CE
- new net !CHG: R7.1, X4.!CHG
- new net !PGOOD: R11.1, X4.!PGOOD
- new net CHARGER_IN: D2.A
- new net ILIM: R3.1, X4.ILIM
- new net ISET: R9.1, X4.ISET
- new net ITERM: R4.1, X4.ITERM
- new net N$1: X4.EN2
- new net N$2: D2.C, X4.IN
- new net THERM: JP8.1, X4.TS
- new net VLIPO: BATT.2, X4.BAT
- net GND: now also BATT.1, JP8.2, R3.2, R4.2, R8.2, R9.2, X4.EN1, X4.TMR, X4.VSS; no longer JP1.1, JP1.10, JP1.3
- net PGOOD: no longer JP1.6
- net VBAT: now also X4.OUT; no longer JP1.4
Other:
- note added: "Batt tmp probe"
- note added: "Battery input"
- moved on the sheet: C1, HP1, HP2, J1, J2, J3, J4, JP4, JP5, R1, R2, SJ1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

Commit message: WeatherChimesv2.6 files from Google Drive
Parts:
- removed BATT: JST 2PH, adafruit:JST_2PIN-SMT-RA
- removed C5, C6: 10uF, adafruit:C-USC0805K
- removed D2: SK34A, microbuilder:DIODE-SCHOTTKYSMA
- removed JP8: (no value), pinhead:PINHD-1X2
- removed R11, R4, R7, R8: 10K, adafruit:R-US_M0805
- removed R3, R9: 1K, adafruit:R-US_M0805
- removed X4: BQ24074, adafruit_power:BQ24074
- added JP1: (no value), microbuilder:HEADER-1X1176MIL
- added U$6, U$7, U$8: MOUNTINGHOLE2.5, microbuilder:MOUNTINGHOLE2.5
Connections:
- removed net !CE: R8.1, X4.!CE
- removed net !CHG: R7.1, X4.!CHG
- removed net !PGOOD: R11.1, X4.!PGOOD
- removed net CHARGER_IN: D2.A
- removed net ILIM: R3.1, X4.ILIM
- removed net ISET: R9.1, X4.ISET
- removed net ITERM: R4.1, X4.ITERM
- removed net N$1: X4.EN2
- removed net N$2: D2.C, X4.IN
- removed net THERM: JP8.1, X4.TS
- removed net VLIPO: BATT.2, X4.BAT
- net GND: now also JP1.1, JP1.10, JP1.3; no longer BATT.1, JP8.2, R3.2, R4.2, R8.2, R9.2, X4.EN1, X4.TMR, X4.VSS
- net PGOOD: now also JP1.6
- net VBAT: now also JP1.4; no longer X4.OUT
Other:
- note added: "SOLAR CHARGER"
- note removed: "Batt tmp probe"
- note removed: "Battery input"
- moved on the sheet: C1, HP1, HP2, J1, J2, J3, J4, JP4, JP5, R1, R2, SJ1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

Commit message: Add files via upload
Other:
- note removed: "SOLAR CHARGER"
Changed lines of the file:
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@@
 <schematic_group name="MS580302BA"/>
 <schematic_group name="LTE_BOARD"/>
+<schematic_group name="SOLAR_CHARGER"/>
 </groups>
 <parts>
@@
 <sheet>
 <plain>
-<text x="83.82" y="-22.86" size="1.778" layer="91">SOLAR CHARGER</text>
 </plain>
 <instances>
@@
 <instance part="U$4" gate="G$1" x="139.7" y="-20.32" smashed="yes"/>
 <instance part="U$5" gate="G$1" x="147.32" y="-20.32" smashed="yes"/>
-<instance part="GND1" gate="1" x="81.28" y="-12.7" smashed="yes">
-<attribute name="VALUE" x="78.74" y="-15.24" size="1.778" layer="96"/>
-</instance>
-<instance part="JP1" gate="G$1" x="91.44" y="-7.62" smashed="yes" rot="R270">
-<attribute name="NAME" x="107.315" y="-1.27" size="1.778" layer="95" rot="R270"/>
-<attribute name="VALUE" x="73.66" y="-1.27" size="1.778" layer="96" rot="R270"/>
-</instance>
-<instance part="GND2" gate="1" x="104.14" y="-15.24" smashed="yes">
-<attribute name="VALUE" x="101.6" y="-17.78" size="1.778" layer="96"/>
-</instance>
-<instance part="GND3" gate="1" x="99.06" y="-15.24" smashed="yes">
-<attribute name="VALUE" x="96.52" y="-17.78" size="1.778" layer="96"/>
+<instance part="GND1" gate="1" x="81.28" y="-2.54" smashed="yes" grouprefs="SOLAR_CHARGER">
+<attribute name="VALUE" x="78.74" y="-5.08" size="1.778" layer="96"/>
+</instance>
+<instance part="JP1" gate="G$1" x="91.44" y="2.54" smashed="yes" rot="R270" grouprefs="SOLAR_CHARGER">
+<attribute name="VALUE" x="73.66" y="8.89" size="1.778" layer="96" rot="R270"/>
+</instance>
+<instance part="GND2" gate="1" x="104.14" y="-5.08" smashed="yes" grouprefs="SOLAR_CHARGER">
+<attribute name="VALUE" x="101.6" y="-7.62" size="1.778" layer="96"/>
+</instance>
+<instance part="GND3" gate="1" x="99.06" y="-5.08" smashed="yes" grouprefs="SOLAR_CHARGER">
+<attribute name="VALUE" x="96.52" y="-7.62" size="1.778" layer="96"/>
 </instance>
 <instance part="GND4" gate="1" x="147.32" y="30.48" smashed="yes" rot="R180">
@@
 </segment>
 <segment>
-<wire x1="81.28" y1="-5.08" x2="81.28" y2="-10.16" width="0.1524" layer="91"/>
+<wire x1="81.28" y1="5.08" x2="81.28" y2="0" width="0.1524" layer="91" grouprefs="SOLAR_CHARGER"/>
 <pinref part="GND1" gate="1" pin="GND"/>
 <pinref part="JP1" gate="G$1" pin="10"/>
@@
 <segment>
 <pinref part="GND2" gate="1" pin="GND"/>
-<wire x1="104.14" y1="-5.08" x2="104.14" y2="-12.7" width="0.1524" layer="91"/>
+<wire x1="104.14" y1="5.08" x2="104.14" y2="-2.54" width="0.1524" layer="91" grouprefs="SOLAR_CHARGER"/>
 <pinref part="JP1" gate="G$1" pin="1"/>
 </segment>
 <segment>
 <pinref part="GND3" gate="1" pin="GND"/>
-<wire x1="99.06" y1="-5.08" x2="99.06" y2="-12.7" width="0.1524" layer="91"/>
+<wire x1="99.06" y1="5.08" x2="99.06" y2="-2.54" width="0.1524" layer="91" grouprefs="SOLAR_CHARGER"/>
 <pinref part="JP1" gate="G$1" pin="3"/>
 </segment>
@@
 <segment>
 <pinref part="JP1" gate="G$1" pin="4"/>
-<wire x1="96.52" y1="-5.08" x2="96.52" y2="-12.7" width="0.1524" layer="91"/>
-<label x="93.98" y="-12.7" size="1.778" layer="95"/>
+<wire x1="96.52" y1="5.08" x2="96.52" y2="-2.54" width="0.1524" layer="91" grouprefs="SOLAR_CHARGER"/>
+<label x="93.98" y="-2.54" size="1.778" layer="95" grouprefs="SOLAR_CHARGER"/>
 </segment>
 <segment>
@@
 <segment>
 <pinref part="JP1" gate="G$1" pin="6"/>
-<wire x1="91.44" y1="-5.08" x2="91.44" y2="-12.7" width="0.1524" layer="91"/>
-<label x="91.44" y="-12.7" size="1.27" layer="95" rot="R270" xref="yes"/>
-</segment>
-<segment>
+<wire x1="91.44" y1="5.08" x2="91.44" y2="-2.54" width="0.1524" layer="91" grouprefs="SOLAR_CHARGER"/>
+<label x="91.44" y="-2.54" size="1.27" layer="95" rot="R270" xref="yes" grouprefs="SOLAR_CHARGER"/>
+</segment>
+<segment>
