File: PCB/Chime/Chime PCB.brd (EAGLE design)
At the start: 102.8 x 78.9 mm, 27 parts, among them U1 MS5803-02BA

Commit message: Add files via upload
Parts:
- removed J5_INT: (no value), SparkFun-Connectors:1X02
- removed JP5_SOLAR: (no value), microbuilder:1X11_ROUND_76
- removed U$13, U$14, U$15, U$16: MOUNTINGHOLE2.5, microbuilder:MOUNTINGHOLE_2.5_PLATED
- added BATT: JST 2PH, adafruit:JST-PH-2-SMT-RA
- added C5, C6: 10uF, adafruit:C0805K
- added D2: SK34A, microbuilder:SMADIODE
- added JP8: (no value), pinhead:1X02
- added R11, R4, R7, R8: 10K, adafruit:M0805
- added R3, R9: 1K, adafruit:M0805
- added X4: BQ24074, adafruit_power:QFN16_3MM
- moved J2_I2C 4.75 mm to (3.30, 39.1)
- moved J6_SPI 4.75 mm to (3.17, 17.4)
- moved J1_I2C 4.75 mm to (3.30, 28.2)
- moved J3_AO 4.75 mm to (3.30, 50.8)
- moved J4_SD1 4.75 mm to (8.26, 61.6)
- moved U$1 2.54 mm to (64.8, 59.7)
Connections:
- new net !CE: R8.1, X4.4
- new net !CHG: R7.1, X4.9
- new net !PGOOD: R11.1, X4.7
- new net CHARGER_IN: D2.A
- new net ILIM: R3.1, X4.12
- new net ISET: R9.1, X4.16
- new net ITERM: R4.1, X4.15
- new net N$1: X4.5
- new net N$2: D2.C, X4.13
- new net THERM: JP8.1, X4.1
- new net VLIPO: BATT.1, X4.2, X4.3
- net A2: no longer J5_INT.1
- net GND: now also BATT.2, JP8.2, R3.2, R4.2, R8.2, R9.2, X4.14, X4.6, X4.8, X4.THERMAL; no longer J5_INT.2, JP5_SOLAR.1, JP5_SOLAR.10, JP5_SOLAR.3
- net PGOOD: no longer JP5_SOLAR.6
- net VBAT: now also X4.10, X4.11; no longer JP5_SOLAR.4
Routing:
- net A2: track 112.9 -> 0.00 mm
- net PGOOD: track 62.3 -> 0.00 mm
- net SCL: track 172.6 -> 127.9 mm
- net MISO: track 96.5 -> 67.6 mm, vias 1 -> 2
- net MOSI: track 93.3 -> 70.2 mm, vias 1 -> 0
- net SCK: track 93.7 -> 73.4 mm
- net SDA: track 154.0 -> 134.2 mm, vias 2 -> 4
- net !PGOOD: track 0.00 -> 16.8 mm
- net N$2: track 0.00 -> 12.5 mm
- net THERM: track 0.00 -> 12.4 mm
- net A0: track 78.3 -> 89.5 mm
- net !CHG: track 0.00 -> 9.98 mm
- net VLIPO: track 0.00 -> 9.59 mm
- net 3VSWITCH: track 72.2 -> 81.4 mm, vias 2 -> 0
- net RX: track 73.0 -> 65.2 mm, vias 0 -> 2
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Other:
- board text added: "SOLAR CHARGER"
- board text added: "Winnie Woo"
- board text removed: "A2"
- board text removed: "CE"
- board text removed: "CHG"
- board text removed: "ISET"
- board text removed: "LIPO"
- board text removed: "OUT"
- board text removed: "PGOOD"
- board text removed: "SOLAR CHARGER this side"
- board text removed: "THERM"
- board text removed: "VBUS"
- board text removed: "Winnie Woo 2023"

Commit message: Add files via upload
Routing:
- net 5VSWITCH: track 63.5 -> 62.1 mm
Changed lines of the file:
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@@
 <contactref element="J8_S5V" pad="1"/>
 <via x="81.661" y="52.324" extent="1-16" drill="0.508"/>
-<wire x1="61.0362" y1="51.57550625" x2="61.73550625" y2="50.8762" width="0.2032" layer="16"/>
 <wire x1="74.41446875" y1="53.3146" x2="75.44553125" y2="53.3146" width="0.2032" layer="16"/>
-<wire x1="52.197" y1="62.865" x2="61.0362" y2="54.0258" width="0.2032" layer="16"/>
+<wire x1="52.197" y1="62.865" x2="64.1858" y2="50.8762" width="0.2032" layer="16"/>
 <wire x1="76.43613125" y1="52.324" x2="81.661" y2="52.324" width="0.2032" layer="16"/>
-<wire x1="61.0362" y1="54.0258" x2="61.0362" y2="51.57550625" width="0.2032" layer="16"/>
 <wire x1="75.44553125" y1="53.3146" x2="76.43613125" y2="52.324" width="0.2032" layer="16"/>
-<wire x1="61.73550625" y1="50.8762" x2="71.97606875" y2="50.8762" width="0.2032" layer="16"/>
+<wire x1="64.1858" y1="50.8762" x2="71.97606875" y2="50.8762" width="0.2032" layer="16"/>
 <wire x1="71.97606875" y1="50.8762" x2="74.41446875" y2="53.3146" width="0.2032" layer="16"/>
 <wire x1="81.661" y1="52.324" x2="81.661" y2="46.11886875" width="0.2032" layer="1"/>

Commit message: Add files via upload
Other:
- board size 102.8 x 78.9 mm -> 101.6 x 78.9 mm
Changed lines of the file:
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@@
 <board>
 <plain>
-<wire x1="-1.27" y1="1.27" x2="101.58" y2="1.27" width="0" layer="20"/>
-<wire x1="101.58" y1="1.27" x2="101.453" y2="80.061" width="0" layer="20"/>
-<wire x1="101.453" y1="80.061" x2="-1.27" y2="80.188" width="0" layer="20"/>
+<wire x1="-1.27" y1="1.27" x2="100.31" y2="1.27" width="0" layer="20"/>
+<wire x1="100.31" y1="1.27" x2="100.183" y2="80.061" width="0" layer="20"/>
+<wire x1="100.183" y1="80.061" x2="-1.27" y2="80.188" width="0" layer="20"/>
 <wire x1="-1.27" y1="80.188" x2="-1.27" y2="1.27" width="0" layer="20"/>
 <dimension x1="-2.54" y1="1.27" x2="-2.54" y2="80.01" x3="-8.89" y3="40.64" textsize="1.778" layer="20" unit="inch"/>
-<dimension x1="-1.27" y1="106.68" x2="101.6" y2="106.68" x3="50.165" y3="83.819996875" textsize="1.778" layer="20" unit="inch"/>
 <dimension x1="26.67" y1="-30.48" x2="-6.35" y2="-30.48" x3="10.16" y3="-27.94" textsize="1.778" layer="47" unit="inch"/>
 <dimension x1="-8.89" y1="-33.02" x2="29.21" y2="-34.29" x3="10.16" y3="-24.003" textsize="1.778" layer="47" dtype="horizontal" unit="inch"/>
@@
 <wire x1="26.67" y1="1.27" x2="26.67" y2="20.32" width="0.2032" layer="21"/>
 <text x="25.654" y="3.429" size="1.27" layer="21" rot="R90">SOLAR CHARGER</text>
+<dimension x1="-1.27" y1="82.55" x2="100.33" y2="82.55" x3="49.53" y3="85.09" textsize="1.778" layer="20" dtype="horizontal" unit="inch"/>
 </plain>
 <attributes>
@@
 <polygon width="0.1524" layer="1">
 <vertex x="-1.27" y="80.01"/>
-<vertex x="101.6" y="80.01"/>
-<vertex x="101.6" y="1.27"/>
+<vertex x="100.33" y="80.01"/>
+<vertex x="100.33" y="1.27"/>
 <vertex x="-1.27" y="1.27"/>
 </polygon>

Commit message: Add files via upload
Parts:
- moved HP1 3.43 mm to (71.5, 62.2)
- moved HP2 3.43 mm to (91.8, 52.1)
- moved U$4 2.54 mm to (95.2, 76.2)
- moved U$5 2.54 mm to (95.2, 5.08)
Routing:
- net RX: track 65.2 -> 58.0 mm
- net MISO: track 67.6 -> 61.7 mm
- net MOSI: track 70.2 -> 74.8 mm
- net 3VSWITCH: track 81.4 -> 77.1 mm
- net VCC: track 155.6 -> 152.2 mm
- net SCL: track 127.9 -> 124.5 mm
- net A1: track 73.7 -> 70.3 mm
- net A0: track 89.5 -> 86.1 mm
- net 5VSWITCH: track 62.1 -> 58.6 mm
- net 4GONOFF: track 60.5 -> 57.1 mm
- net SDA: track 134.2 -> 130.7 mm
- net TX: track 59.4 -> 56.1 mm
- net 5VRAIL: track 47.9 -> 46.1 mm
- net VBAT: track 96.9 -> 95.4 mm
- net SCK: track 73.4 -> 72.8 mm
Other:
- board size 101.6 x 78.9 mm -> 100.3 x 78.9 mm

Commit message: Add files via upload
Other:
- board size 100.3 x 78.9 mm -> 99 x 78.9 mm
Changed lines of the file:
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@@
 <board>
 <plain>
-<wire x1="-1.27" y1="1.27" x2="99.04" y2="1.27" width="0" layer="20"/>
+<wire x1="0" y1="1.27" x2="99.04" y2="1.27" width="0" layer="20"/>
 <wire x1="99.04" y1="1.27" x2="98.913" y2="80.061" width="0" layer="20"/>
-<wire x1="98.913" y1="80.061" x2="-1.27" y2="80.188" width="0" layer="20"/>
-<wire x1="-1.27" y1="80.188" x2="-1.27" y2="1.27" width="0" layer="20"/>
+<wire x1="98.913" y1="80.061" x2="0" y2="80.188" width="0" layer="20"/>
+<wire x1="0" y1="80.188" x2="0" y2="1.27" width="0" layer="20"/>
 <dimension x1="-2.54" y1="1.27" x2="-2.54" y2="80.01" x3="-8.89" y3="40.64" textsize="1.778" layer="20" unit="inch"/>
 <dimension x1="26.67" y1="-30.48" x2="-6.35" y2="-30.48" x3="10.16" y3="-27.94" textsize="1.778" layer="47" unit="inch"/>
@@
 <wire x1="26.67" y1="1.27" x2="26.67" y2="20.32" width="0.2032" layer="21"/>
 <text x="25.654" y="3.429" size="1.27" layer="21" rot="R90">SOLAR CHARGER</text>
-<dimension x1="-1.27" y1="81.28" x2="99.06" y2="81.28" x3="48.895" y3="82.55" textsize="1.778" layer="20" unit="inch"/>
 <wire x1="87.122" y1="10.541" x2="92.075" y2="10.541" width="0.2032" layer="25" curve="-180"/>
 <circle x="89.662" y="13.589" radius="0.523634375" width="0.2032" layer="25"/>
@@
 <wire x1="87.122" y1="10.541" x2="92.075" y2="10.541" width="0.2032" layer="25"/>
 <circle x="89.662" y="13.589" radius="0.523634375" width="0.2032" layer="25"/>
+<dimension x1="0" y1="82.55" x2="99.06" y2="82.55" x3="49.53" y3="83.82" textsize="1.778" layer="20" unit="inch"/>
 </plain>
 <attributes>
@@
 <contactref element="U$1" pad="GND3"/>
 <polygon width="0.1524" layer="1">
-<vertex x="-1.27" y="80.01"/>
+<vertex x="0" y="80.01"/>
 <vertex x="99.06" y="80.01"/>
 <vertex x="99.06" y="1.27"/>
-<vertex x="-1.27" y="1.27"/>
+<vertex x="0" y="1.27"/>
 </polygon>
 <contactref element="HP1" pad="4"/>
