File: PCB/Chime/Chime PCB.brd (EAGLE design)
At the start: 99 x 78.9 mm, 33 parts, among them U1 MS5803-02BA, X4 BQ24074

Commit message: Add files via upload
Parts:
- removed J1_I2C: (no value), SparkFun-Connectors:1X04
- removed J3_AO, J4_SD1: (no value), SparkFun-Connectors:1X03
- removed J6_SPI: (no value), SparkFun-Connectors:1X06_LOCK
- added J1_SPI: 1725698, 1725698:1725698
- added J4_A1, J5_A0: 1725669, 1725669:1725669
- added J6_TSL2591: (no value), SparkFun-Connectors:1X06_LOCK
- added JP9: (no value), pinhead:1X02
- added U$17, U$19: MOUNTINGHOLE2.5, microbuilder:MOUNTINGHOLE_2.5_PLATED
- J2_I2C: value (none) -> 1725672; device SparkFun-Connectors:1X04 -> 1725672:1725672
- U$1: device LTE_BOARD:LTE_BOARD_FOOTPRINT -> LTE_BOARD_LOOM:LTE_BOARD_FOOTPRINT
- moved HP1 72.7 mm to (16.6, 14.6), turned to 0 degrees
- moved HP2 67.2 mm to (26.8, 34.9), turned to 0 degrees
- moved JP8 48.7 mm to (2.54, 34.3), turned to 270 degrees
- moved U$1 45.7 mm to (19.1, 58.4), turned to 180 degrees
- moved JP4 45.1 mm to (41.0, 18.8), turned to 90 degrees
- moved BATT 43.3 mm to (10.2, 27.4), turned to 90 degrees
- moved R1 40.2 mm to (48.9, 20.1), turned to 0 degrees
- moved C1 39.4 mm to (38.2, 24.9), turned to 90 degrees
- moved R9 38.4 mm to (14.2, 35.7), turned to 90 degrees
- moved J2_I2C 38.3 mm to (30.5, 66.0)
- moved R4 37.6 mm to (16.1, 37.1), turned to 90 degrees
- moved J7_S3V 37.4 mm to (22.4, 46.7), turned to 180 degrees
- moved U$4 36.7 mm to (58.5, 74.8)
- moved U$5 36.7 mm to (58.5, 3.68)
- moved U1 36.2 mm to (42.8, 24.9), turned to 90 degrees
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Connections:
- removed net A4: J6_SPI.3
- new net INT: J6_TSL2591.6
- new net VIN: J6_TSL2591.1
- net A0: now also J5_A0.2; no longer J4_SD1.2
- net A1: now also J4_A1.2; no longer J3_AO.2
- net A3: now also J1_SPI.3
- net CHARGER_IN: now also JP9.1
- net GND: now also C5.2, C6.2, J1_SPI.2, J4_A1.3, J5_A0.3, J6_TSL2591.3; no longer J1_I2C.2, J3_AO.3, J4_SD1.3, J6_SPI.2
- net MISO: now also J1_SPI.6; no longer J6_SPI.6
- net MOSI: now also J1_SPI.5; no longer J6_SPI.5
- net SCK: now also J1_SPI.4; no longer J6_SPI.4
- net SCL: now also J6_TSL2591.4; no longer J1_I2C.3
- net SDA: now also J6_TSL2591.5; no longer J1_I2C.4
- net VCC: now also J1_SPI.1, J4_A1.1, J5_A0.1, J6_TSL2591.2; no longer J1_I2C.1, J3_AO.1, J4_SD1.1, J6_SPI.1
- net VLIPO: now also C5.1, C6.1
Routing:
- net VBAT: track 95.4 -> 7.59 mm, vias 1 -> 2
- net SCL: track 124.5 -> 50.2 mm
- net SDA: track 130.7 -> 68.1 mm, vias 4 -> 1
- net A3: track 0.00 -> 62.0 mm
- net 4GONOFF: track 57.1 -> 5.44 mm
- net TX: track 56.1 -> 4.50 mm, vias 1 -> 0
- net RX: track 58.0 -> 9.96 mm, vias 2 -> 0
- net 3VSWITCH: track 77.1 -> 33.9 mm, vias 0 -> 2
- net VCC: track 152.2 -> 189.4 mm, vias 0 -> 1
- net A0: track 86.1 -> 59.4 mm, vias 1 -> 0
- net 5VSWITCH: track 58.6 -> 33.4 mm, vias 1 -> 2
- net 5VRAIL: track 46.1 -> 24.6 mm
- net N$2: track 12.5 -> 27.8 mm, vias 0 -> 2
- net A1: track 70.3 -> 55.2 mm, vias 1 -> 0
- net !PGOOD: track 16.8 -> 2.61 mm
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Other:
- board size 99 x 78.9 mm -> 62.2 x 77.6 mm
- board text added: "A3"
- board text added: "Chime V1"
- board text added: "LTE board this side"
- board text removed: "0x76 Def"
- board text removed: "A4"
- board text removed: "AO"
- board text removed: "Chime"
- board text removed: "I2C"
- board text removed: "LTE BOARD this side"
- board text removed: "OPEnS"
- board text removed: "SDI"
- board text removed: "SOLAR CHARGER"
- board text removed: "SPI"

Commit message: Add files via upload
Routing:
- net VCC: track 189.4 -> 178.1 mm
Changed lines of the file:
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@@
 <wire x1="45.212" y1="24.257" x2="47.117" y2="22.352" width="0.2032" layer="1"/>
 <wire x1="49.784" y1="20.127" x2="49.845" y2="20.066" width="0.2032" layer="1"/>
-<wire x1="41.36435" y1="25.1206" x2="45.50485" y2="25.1206" width="0.2032" layer="1"/>
+<wire x1="45.50485" y1="25.1206" x2="41.36435" y2="25.1206" width="0.2032" layer="1"/>
 <contactref element="J1_SPI" pad="1"/>
 <contactref element="J2_I2C" pad="1"/>
@@
 <wire x1="50.165" y1="24.511" x2="50.165" y2="28.448" width="0.2032" layer="1"/>
 <wire x1="50.165" y1="28.448" x2="49.9415" y2="28.6715" width="0.2032" layer="1"/>
-<wire x1="49.784" y1="20.84145" x2="49.784" y2="20.32" width="0.2032" layer="1"/>
 <wire x1="49.784" y1="20.32" x2="49.784" y2="20.127" width="0.2032" layer="1"/>
-<wire x1="45.50485" y1="25.1206" x2="49.784" y2="20.84145" width="0.2032" layer="1"/>
-<wire x1="50.165" y1="23.50845" x2="50.165" y2="24.511" width="0.2032" layer="1"/>
 <wire x1="47.117" y1="22.352" x2="49.00855" y2="22.352" width="0.2032" layer="1"/>
-<wire x1="49.00855" y1="22.352" x2="50.165" y2="23.50845" width="0.2032" layer="1"/>
-<wire x1="51.242" y1="21.778" x2="49.784" y2="20.32" width="0.2032" layer="1"/>
+<wire x1="51.242" y1="21.778" x2="50.038" y2="20.574" width="0.2032" layer="1"/>
+<wire x1="50.038" y1="20.574" x2="49.784" y2="20.32" width="0.2032" layer="1"/>
 <wire x1="49.972" y1="28.702" x2="51.242" y2="27.432" width="0.2032" layer="1"/>
 <wire x1="51.242" y1="27.432" x2="51.242" y2="21.778" width="0.2032" layer="1"/>
@@
 <wire x1="40.7416" y1="34.40946875" x2="40.7416" y2="38.9636" width="0.2032" layer="1"/>
 <wire x1="40.1442" y1="26.34075" x2="40.1442" y2="33.81206875" width="0.2032" layer="1"/>
-<wire x1="49.59275" y1="23.5712" x2="47.68925" y2="23.5712" width="0.2032" layer="1"/>
-<wire x1="49.7713" y1="23.74975" x2="49.59275" y2="23.5712" width="0.2032" layer="1"/>
 <wire x1="41.36435" y1="25.1206" x2="40.1442" y2="26.34075" width="0.2032" layer="1"/>
-<wire x1="46.13985" y1="25.1206" x2="45.50485" y2="25.1206" width="0.2032" layer="1"/>
-<wire x1="47.68925" y1="23.5712" x2="46.13985" y2="25.1206" width="0.2032" layer="1"/>
-<wire x1="49.972" y1="28.702" x2="49.7713" y2="28.5013" width="0.2032" layer="1"/>
-<wire x1="49.7713" y1="28.5013" x2="49.7713" y2="23.74975" width="0.2032" layer="1"/>
 <via x="50.8" y="31.75" extent="1-16" drill="0.508"/>
 <wire x1="41.402" y1="40.513" x2="45.8724" y2="36.0426" width="0.2032" layer="16"/>
@@
 <wire x1="50.8" y1="31.75" x2="50.8" y2="29.53" width="0.2032" layer="1"/>
 <wire x1="50.8" y1="29.53" x2="49.972" y2="28.702" width="0.2032" layer="1"/>
+<wire x1="49.00855" y1="22.352" x2="50.038" y2="21.32255" width="0.2032" layer="1"/>
+<wire x1="50.038" y1="21.32255" x2="50.038" y2="20.574" width="0.2032" layer="1"/>
+<wire x1="42.6942" y1="23.44325" x2="42.87275" y2="23.6218" width="0.2032" layer="1"/>
+<wire x1="45.0848" y1="23.6218" x2="45.72" y2="24.257" width="0.2032" layer="1"/>
+<wire x1="42.149" y1="22.192" x2="42.6942" y2="22.7372" width="0.2032" layer="1"/>
+<wire x1="42.6942" y1="22.7372" x2="42.6942" y2="23.44325" width="0.2032" layer="1"/>
+<wire x1="42.87275" y1="23.6218" x2="45.0848" y2="23.6218" width="0.2032" layer="1"/>
+<wire x1="45.72" y1="24.257" x2="45.72" y2="24.90545" width="0.2032" layer="1"/>
+<wire x1="45.72" y1="24.90545" x2="45.50485" y2="25.1206" width="0.2032" layer="1"/>
 </signal>
 <signal name="RX">

Commit message: Add files via upload
Parts:
- J4_A1, J5_A0: value 1725669 -> 282834-3; device 1725669:1725669 -> Fixed Terminal Blocks 3P:TE_282834-3
- moved D2 9.83 mm to (13.2, 24.3), turned to 270 degrees
- moved JP9 9.49 mm to (3.43, 16.1), turned to 270 degrees
- moved BATT 6.34 mm to (4.83, 24.0)
- moved J5_A0 5.08 mm to (5.08, 66.0), turned to 0 degrees
- moved J4_A1 5.08 mm to (17.8, 66.0), turned to 0 degrees
- moved J8_S5V 4.02 mm to (18.4, 51.7)
- moved J7_S3V 4.02 mm to (18.5, 45.5)
- moved J6_TSL2591 1.78 mm to (40.6, 40.6)
- moved JP8 1.20 mm to (2.92, 35.4)
- moved U$17 0.13 mm to (57.1, 53.2)
- turned R8 to 270 degrees
Connections:
- net GND: now also J4_A1.1, J5_A0.1; no longer J4_A1.3, J5_A0.3
- net VCC: now also J4_A1.3, J5_A0.3; no longer J4_A1.1, J5_A0.1
Routing:
- net N$2: track 27.8 -> 14.3 mm
- net VLIPO: track 7.73 -> 15.8 mm, vias 0 -> 2
- net CHARGER_IN: track 8.60 -> 13.9 mm
- net 5VSWITCH: track 33.4 -> 36.7 mm
- net 3VSWITCH: track 33.9 -> 37.2 mm
- net A3: track 62.0 -> 65.1 mm
- net A0: track 59.4 -> 61.7 mm
- net !CE: track 0.00 -> 2.14 mm
- net A1: track 55.2 -> 57.3 mm
- net 5VRAIL: track 24.6 -> 26.7 mm
- net VCC: track 178.1 -> 177.5 mm

Commit message: Add files via upload
Parts:
- moved J7_S3V 7.73 mm to (17.3, 53.1)
- moved J8_S5V 5.24 mm to (17.1, 46.6)
Routing:
- net 3VSWITCH: track 37.2 -> 41.3 mm, vias 2 -> 1
- net A0: track 61.7 -> 59.6 mm
- net SDA: track 68.1 -> 66.5 mm
- net 5VSWITCH: track 36.7 -> 35.6 mm, vias 2 -> 1
- net A3: track 65.1 -> 64.2 mm
- net VCC: track 177.5 -> 178.1 mm, vias 1 -> 2
- net SCK: track 70.3 -> 69.6 mm
- net A1: track 57.3 -> 57.8 mm
Other:
- board text added: "0x76 Def"
- board text added: "Chime"
- board text removed: "Chime V1"
