File: PCB/Chime v2/Chime PCB v2.sch (EAGLE design)
At the start: 34 parts, among them J1_I2C1 1725672, J2_I2C 1725672, J4_A1 282834-3, J5_A0 282834-3, U1 MS5803-02BA, X4 BQ24074

Commit message: Add files via upload
Parts:
- removed J1_I2C1: 1725672, 1725672:1725672
- removed J6_TSL2591: (no value), SparkFun-Connectors:CONN_06LOCK
- removed J7_S3V, J8_S5V: (no value), SparkFun-Connectors:CONN_02
- added J1_SPI: 1725698, 1725698:1725698
Connections:
- removed net INT: J6_TSL2591.6
- removed net VIN: J6_TSL2591.1
- net 3VSWITCH: no longer J7_S3V.1
- net 5VSWITCH: no longer J8_S5V.1
- net A3: now also J1_SPI.3
- net GND: now also J1_SPI.2; no longer J1_I2C1.2, J6_TSL2591.3, J7_S3V.2, J8_S5V.2
- net MISO: now also J1_SPI.6
- net MOSI: now also J1_SPI.5
- net SCK: now also J1_SPI.4
- net SCL: no longer J1_I2C1.3, J6_TSL2591.4
- net SDA: no longer J1_I2C1.4, J6_TSL2591.5
- net VCC: now also J1_SPI.1; no longer J1_I2C1.1, J6_TSL2591.2
Changed lines of the file:
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@@
 <part name="D2" library="microbuilder" deviceset="DIODE-SCHOTTKY" device="SMA" value="SK34A"/>
 <part name="GND1" library="supply1" library_urn="urn:adsk.eagle:library:371" deviceset="GND" device=""/>
-<part name="J6_TSL2591" library="SparkFun-Connectors" deviceset="CONN_06" device="LOCK"/>
 <part name="J2_I2C" library="1725672" deviceset="1725672" device=""/>
-<part name="J7_S3V" library="SparkFun-Connectors" deviceset="CONN_02" device=""/>
-<part name="J8_S5V" library="SparkFun-Connectors" deviceset="CONN_02" device=""/>
+<part name="J1_SPI" library="1725698" deviceset="1725698" device=""/>
 <part name="SJ1" library="SparkFun-Jumpers" library_urn="urn:adsk.eagle:library:528" deviceset="JUMPER-SMT_3_1-NC_TRACE" device="_SILK" package3d_urn="urn:adsk.eagle:package:39288/1"/>
 <part name="J4_A1" library="Fixed Terminal Blocks 3P" deviceset="282834-3" device=""/>
 <part name="J5_A0" library="Fixed Terminal Blocks 3P" deviceset="282834-3" device=""/>
-<part name="J1_I2C1" library="1725672" deviceset="1725672" device=""/>
 </parts>
 <sheets>
@@
 <attribute name="VALUE" x="55.88" y="40.64" size="1.778" layer="96" rot="R270"/>
 </instance>
-<instance part="J6_TSL2591" gate="JP1" x="274.32" y="93.98" smashed="yes">
-<attribute name="VALUE" x="269.24" y="84.074" size="1.778" layer="96" font="vector"/>
-<attribute name="NAME" x="269.24" y="104.648" size="1.778" layer="95" font="vector"/>
-</instance>
 <instance part="J2_I2C" gate="G$1" x="312.674" y="62.484" smashed="yes" rot="R180">
 <attribute name="NAME" x="303.784" y="75.184" size="1.778" layer="95" rot="R180" align="center-left"/>
 </instance>
-<instance part="J7_S3V" gate="G$1" x="353.06" y="63.5" smashed="yes">
-<attribute name="VALUE" x="350.52" y="58.674" size="1.778" layer="96" font="vector"/>
-<attribute name="NAME" x="350.52" y="69.088" size="1.778" layer="95" font="vector"/>
-</instance>
-<instance part="J8_S5V" gate="G$1" x="353.06" y="78.74" smashed="yes">
-<attribute name="VALUE" x="350.52" y="73.914" size="1.778" layer="96" font="vector"/>
-<attribute name="NAME" x="350.52" y="84.328" size="1.778" layer="95" font="vector"/>
+<instance part="J1_SPI" gate="G$1" x="281.94" y="60.96" smashed="yes" rot="R180">
+<attribute name="NAME" x="273.812" y="78.486" size="1.778" layer="95" rot="R180" align="center-left"/>
 </instance>
 <instance part="SJ1" gate="G$1" x="127" y="127" smashed="yes" grouprefs="MS580302BA">
@@
 <instance part="J5_A0" gate="G$1" x="330.2" y="78.74" smashed="yes">
 <attribute name="NAME" x="327.40435" y="84.331309375" size="1.0166" layer="95"/>
-</instance>
-<instance part="J1_I2C1" gate="G$1" x="284.734" y="62.484" smashed="yes" rot="R180">
-<attribute name="NAME" x="275.844" y="75.184" size="1.778" layer="95" rot="R180" align="center-left"/>
 </instance>
 </instances>
@@
 </segment>
 <segment>
+<pinref part="J1_SPI" gate="G$1" pin="2"/>
+<wire x1="281.94" y1="63.5" x2="289.56" y2="63.5" width="0.1524" layer="91"/>
+<label x="287.02" y="63.5" size="1.778" layer="95"/>
+</segment>
+<segment>
 <pinref part="J2_I2C" gate="G$1" pin="2"/>
 <wire x1="312.674" y1="65.024" x2="318.262" y2="65.024" width="0.1524" layer="91"/>
@@
 </segment>
 <segment>
-<pinref part="J6_TSL2591" gate="JP1" pin="3"/>
-<wire x1="279.4" y1="93.98" x2="287.02" y2="93.98" width="0.1524" layer="91"/>
-<label x="281.94" y="93.98" size="1.778" layer="95"/>
-</segment>
-<segment>
-<pinref part="J8_S5V" gate="G$1" pin="2"/>
-<wire x1="360.68" y1="81.28" x2="368.3" y2="81.28" width="0.1524" layer="91"/>
-<label x="363.22" y="81.28" size="1.778" layer="95"/>
-</segment>
-<segment>
-<pinref part="J7_S3V" gate="G$1" pin="2"/>
-<wire x1="360.68" y1="66.04" x2="368.3" y2="66.04" width="0.1524" layer="91"/>
-<label x="363.22" y="66.04" size="1.778" layer="95"/>
-</segment>
-<segment>
 <pinref part="C6" gate="G$1" pin="2"/>
 <pinref part="GND23" gate="1" pin="GND"/>
@@
 <wire x1="335.28" y1="81.28" x2="340.36" y2="81.28" width="0.1524" layer="91"/>
 <label x="337.82" y="81.28" size="1.778" layer="95"/>
-</segment>
-<segment>
-<pinref part="J1_I2C1" gate="G$1" pin="2"/>
-<wire x1="284.734" y1="65.024" x2="290.322" y2="65.024" width="0.1524" layer="91"/>
-<label x="287.528" y="65.024" size="1.778" layer="95"/>
 </segment>
 </net>
@@
 </segment>
 <segment>
+<pinref part="J1_SPI" gate="G$1" pin="1"/>
+<wire x1="281.94" y1="60.96" x2="289.56" y2="60.96" width="0.1524" layer="91"/>
+<label x="287.02" y="60.96" size="1.778" layer="95"/>
+</segment>
+<segment>
 <pinref part="J2_I2C" gate="G$1" pin="1"/>
 <wire x1="312.674" y1="62.484" x2="318.262" y2="62.484" width="0.1524" layer="91"/>
@@
 </segment>
 <segment>
-<pinref part="J6_TSL2591" gate="JP1" pin="2"/>
-<wire x1="279.4" y1="91.44" x2="287.02" y2="91.44" width="0.1524" layer="91"/>
-<label x="281.94" y="91.44" size="1.778" layer="95"/>
-</segment>
-<segment>
 <pinref part="J4_A1" gate="G$1" pin="3"/>
 <wire x1="335.28" y1="60.96" x2="340.36" y2="60.96" width="0.1524" layer="91"/>
@@
 <label x="337.82" y="76.2" size="1.778" layer="95"/>
 </segment>
-<segment>
-<pinref part="J1_I2C1" gate="G$1" pin="1"/>
-<wire x1="284.734" y1="62.484" x2="290.322" y2="62.484" width="0.1524" layer="91"/>
-<label x="287.528" y="62.484" size="1.778" layer="95"/>
-</segment>
 </net>
 <net name="A1" class="0">
@@
 <label x="177.8" y="119.38" size="1.27" layer="95" rot="R180" xref="yes" grouprefs="HYPNOS"/>
 </segment>
+<segment>
+<pinref part="J1_SPI" gate="G$1" pin="3"/>
+<wire x1="281.94" y1="66.04" x2="289.56" y2="66.04" width="0.1524" layer="91"/>
+<label x="287.02" y="66.04" size="1.778" layer="95"/>
+</segment>
 </net>
 <net name="SCK" class="0">
@@
 <label x="177.8" y="111.76" size="1.27" layer="95" rot="R180" xref="yes" grouprefs="HYPNOS"/>
 </segment>
+<segment>
+<pinref part="J1_SPI" gate="G$1" pin="4"/>
+<wire x1="281.94" y1="68.58" x2="289.56" y2="68.58" width="0.1524" layer="91"/>
+<label x="287.02" y="68.58" size="1.778" layer="95"/>
+</segment>
 </net>
 <net name="MOSI" class="0">
@@
 <label x="177.8" y="109.22" size="1.27" layer="95" rot="R180" xref="yes" grouprefs="HYPNOS"/>
 </segment>
+<segment>
+<pinref part="J1_SPI" gate="G$1" pin="5"/>
+<wire x1="281.94" y1="71.12" x2="289.56" y2="71.12" width="0.1524" layer="91"/>
+<label x="287.02" y="71.12" size="1.778" layer="95"/>
+</segment>
 </net>
 <net name="MISO" class="0">
@@
 <wire x1="182.88" y1="106.68" x2="177.8" y2="106.68" width="0.1524" layer="91" grouprefs="HYPNOS"/>
 <label x="177.8" y="106.68" size="1.27" layer="95" rot="R180" xref="yes" grouprefs="HYPNOS"/>
+</segment>
+<segment>
+<pinref part="J1_SPI" gate="G$1" pin="6"/>
+<wire x1="281.94" y1="73.66" x2="289.56" y2="73.66" width="0.1524" layer="91"/>
+<label x="287.02" y="73.66" size="1.778" layer="95"/>
 </segment>
 </net>
@@
 <wire x1="312.674" y1="70.104" x2="318.008" y2="70.104" width="0.1524" layer="91"/>
 <label x="315.468" y="70.358" size="1.778" layer="95"/>
-</segment>
-<segment>
-<pinref part="J6_TSL2591" gate="JP1" pin="5"/>
-<wire x1="279.4" y1="99.06" x2="287.02" y2="99.06" width="0.1524" layer="91"/>
-<label x="281.94" y="99.06" size="1.778" layer="95"/>
-</segment>
-<segment>
-<pinref part="J1_I2C1" gate="G$1" pin="4"/>
-<wire x1="284.734" y1="70.104" x2="290.068" y2="70.104" width="0.1524" layer="91"/>
-<label x="287.528" y="70.358" size="1.778" layer="95"/>
 </segment>
 </net>
@@
 <label x="315.468" y="67.564" size="1.778" layer="95"/>
 </segment>
-<segment>
-<pinref part="J6_TSL2591" gate="JP1" pin="4"/>
-<wire x1="279.4" y1="96.52" x2="287.02" y2="96.52" width="0.1524" layer="91"/>
-<label x="281.94" y="96.52" size="1.778" layer="95"/>
-</segment>
-<segment>
-<pinref part="J1_I2C1" gate="G$1" pin="3"/>
-<wire x1="284.734" y1="67.564" x2="290.322" y2="67.564" width="0.1524" layer="91"/>
-<label x="287.528" y="67.564" size="1.778" layer="95"/>
-</segment>
 </net>
 <net name="EN" class="0">
@@
 <label x="213.36" y="111.76" size="1.27" layer="95" rot="R180" xref="yes" grouprefs="HYPNOS"/>
 </segment>
-<segment>
-<pinref part="J8_S5V" gate="G$1" pin="1"/>
-<wire x1="360.68" y1="78.74" x2="368.3" y2="78.74" width="0.1524" layer="91"/>
-<label x="363.22" y="78.74" size="1.778" layer="95"/>
-</segment>
 </net>
 <net name="3VSWITCH" class="0">
@@
 <wire x1="220.98" y1="109.22" x2="213.36" y2="109.22" width="0.1524" layer="91" grouprefs="HYPNOS"/>
 <label x="213.36" y="109.22" size="1.27" layer="95" rot="R180" xref="yes" grouprefs="HYPNOS"/>
-</segment>
-<segment>
-<pinref part="J7_S3V" gate="G$1" pin="1"/>
-<wire x1="360.68" y1="63.5" x2="368.3" y2="63.5" width="0.1524" layer="91"/>
-<label x="363.22" y="63.5" size="1.778" layer="95"/>
 </segment>
 </net>
@@
 </segment>
 </net>
-<net name="INT" class="0">
-<segment>
-<pinref part="J6_TSL2591" gate="JP1" pin="6"/>
-<wire x1="279.4" y1="101.6" x2="287.02" y2="101.6" width="0.1524" layer="91"/>
-<label x="281.94" y="101.6" size="1.778" layer="95"/>
-</segment>
-</net>
-<net name="VIN" class="0">
-<segment>
-<pinref part="J6_TSL2591" gate="JP1" pin="1"/>
-<wire x1="279.4" y1="88.9" x2="287.02" y2="88.9" width="0.1524" layer="91"/>
-<label x="281.94" y="88.9" size="1.778" layer="95"/>
-</segment>
-</net>
