File: PCB/Chime v2/Chime PCB v2_511.brd (EAGLE design)
At the start: 64.8 x 68.6 mm, 33 parts, among them J1_SPI 1725698, J2_I2C 1725672, J4_A1 282834-3, J5_A0 282834-3, U1 MS5803-02BA, X4 BQ24074

Commit message: Added LEDs
Routing:
- net VBAT: track 8.09 -> 43.3 mm, vias 2 -> 5
- net N$5: track 0.00 -> 30.2 mm
- net N$4: track 0.00 -> 23.9 mm
- net VCC: track 164.5 -> 152.3 mm, vias 0 -> 1
- net A3: track 51.0 -> 41.2 mm
- net A1: track 46.1 -> 42.9 mm
- net 5VRAIL: track 51.4 -> 52.4 mm
Other:
- board text added: "Chime v2.2"
- board text removed: "Chime v2.1"

Commit message: GND Air Wires
Routing:
- net GND: track 19.8 -> 228.4 mm, vias 2 -> 7
- net N$2: track 13.9 -> 15.0 mm
Changed lines of the file:
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@@
 <vertex x="-1.27" y="-1.27"/>
 </polygon>
-<wire x1="18.693" y1="32.127" x2="18.7482" y2="32.0718" width="0.2032" layer="1"/>
-<wire x1="18.7482" y1="32.0718" x2="19.21925" y2="32.0718" width="0.2032" layer="1"/>
-<wire x1="19.41405" y1="31.877" x2="20.193" y2="31.877" width="0.2032" layer="1"/>
-<wire x1="19.21925" y1="32.0718" x2="19.41405" y2="31.877" width="0.2032" layer="1"/>
 <wire x1="20.193" y1="31.877" x2="20.443" y2="31.627" width="0.2032" layer="1"/>
 <wire x1="20.443" y1="31.627" x2="21.693" y2="31.627" width="0.2032" layer="1"/>
@@
 <wire x1="46.99" y1="22.815675" x2="46.0502" y2="21.875875" width="0.2032" layer="16"/>
 <contactref element="JP9" pad="2"/>
+<wire x1="14.224" y1="36.637" x2="15.748" y2="38.161" width="0.2032" layer="1"/>
+<wire x1="15.748" y1="38.161" x2="16.256" y2="38.161" width="0.2032" layer="1"/>
+<wire x1="3.81" y1="49.53" x2="4.47644375" y2="49.53" width="0.2032" layer="1"/>
+<wire x1="10.76355625" y1="49.53" x2="16.51" y2="49.53" width="0.2032" layer="1"/>
+<wire x1="4.47644375" y1="49.53" x2="5.80124375" y2="50.8548" width="0.2032" layer="1"/>
+<wire x1="5.80124375" y1="50.8548" x2="9.43875625" y2="50.8548" width="0.2032" layer="1"/>
+<wire x1="9.43875625" y1="50.8548" x2="10.76355625" y2="49.53" width="0.2032" layer="1"/>
+<wire x1="16.51" y1="49.53" x2="17.17644375" y2="49.53" width="0.2032" layer="16"/>
+<wire x1="31.35065" y1="49.53" x2="31.75" y2="49.53" width="0.2032" layer="16"/>
+<wire x1="17.17644375" y1="49.53" x2="18.50124375" y2="50.8548" width="0.2032" layer="16"/>
+<wire x1="18.50124375" y1="50.8548" x2="30.02585" y2="50.8548" width="0.2032" layer="16"/>
+<wire x1="30.02585" y1="50.8548" x2="31.35065" y2="49.53" width="0.2032" layer="16"/>
+<wire x1="31.75" y1="49.53" x2="32.650075" y2="49.53" width="0.2032" layer="16"/>
+<wire x1="46.59065" y1="49.53" x2="46.99" y2="49.53" width="0.2032" layer="16"/>
+<wire x1="32.650075" y1="49.53" x2="33.809675" y2="50.6896" width="0.2032" layer="16"/>
+<wire x1="45.43105" y1="50.6896" x2="46.59065" y2="49.53" width="0.2032" layer="16"/>
+<wire x1="33.809675" y1="50.6896" x2="45.43105" y2="50.6896" width="0.2032" layer="16"/>
+<wire x1="31.75" y1="58.42" x2="31.75" y2="49.53" width="0.2032" layer="16"/>
+<wire x1="17.526" y1="26.559" x2="19.685" y2="26.559" width="0.2032" layer="1"/>
+<wire x1="19.685" y1="26.559" x2="21.794" y2="26.559" width="0.2032" layer="1"/>
+<wire x1="21.794" y1="26.559" x2="21.844" y2="26.609" width="0.2032" layer="1"/>
+<wire x1="48.133" y1="24.511" x2="47.752" y2="24.13" width="0.2032" layer="1"/>
+<wire x1="47.752" y1="24.13" x2="46.99" y2="24.13" width="0.2032" layer="1"/>
+<wire x1="43.449" y1="27.592" x2="43.815" y2="27.958" width="0.2032" layer="1"/>
+<wire x1="43.815" y1="27.958" x2="43.815" y2="30.353" width="0.2032" layer="1"/>
+<wire x1="40.32275" y1="29.0218" x2="40.1442" y2="28.84325" width="0.2032" layer="1"/>
+<wire x1="40.1442" y1="28.84325" x2="40.1442" y2="26.34075" width="0.2032" layer="1"/>
+<wire x1="45.9994" y1="25.1206" x2="46.99" y2="24.13" width="0.2032" layer="1"/>
+<wire x1="42.9038" y1="28.83825" x2="42.72025" y2="29.0218" width="0.2032" layer="1"/>
+<wire x1="42.72025" y1="29.0218" x2="40.32275" y2="29.0218" width="0.2032" layer="1"/>
+<wire x1="40.1442" y1="26.34075" x2="41.36435" y2="25.1206" width="0.2032" layer="1"/>
+<wire x1="41.36435" y1="25.1206" x2="45.9994" y2="25.1206" width="0.2032" layer="1"/>
+<wire x1="43.449" y1="27.592" x2="42.9038" y2="28.1372" width="0.2032" layer="1"/>
+<wire x1="42.9038" y1="28.1372" x2="42.9038" y2="28.83825" width="0.2032" layer="1"/>
+<wire x1="38.227" y1="25.842" x2="38.227" y2="28.067" width="0.2032" layer="1"/>
+<wire x1="38.227" y1="28.067" x2="40.64" y2="30.48" width="0.2032" layer="1"/>
+<wire x1="40.64" y1="30.48" x2="43.688" y2="30.48" width="0.2032" layer="1"/>
+<wire x1="43.688" y1="30.48" x2="43.815" y2="30.353" width="0.2032" layer="1"/>
+<wire x1="24.257" y1="14.605" x2="20.32" y2="18.542" width="0.2032" layer="16"/>
+<wire x1="20.32" y1="18.542" x2="20.32" y2="19.05" width="0.2032" layer="16"/>
+<via x="20.32" y="19.05" extent="1-16" drill="0.508"/>
+<wire x1="20.32" y1="19.05" x2="21.844" y2="20.574" width="0.2032" layer="1"/>
+<wire x1="21.844" y1="20.574" x2="21.844" y2="26.609" width="0.2032" layer="1"/>
+<wire x1="8.526" y1="23.003" x2="8.7795" y2="22.7495" width="0.2032" layer="1"/>
+<wire x1="8.7795" y1="22.7495" x2="10.16" y2="21.369" width="0.2032" layer="1"/>
+<wire x1="10.16" y1="21.369" x2="10.16" y2="17.78" width="0.2032" layer="1"/>
+<wire x1="4.70473125" y1="18.5166" x2="2.15326875" y2="18.5166" width="0.2032" layer="1"/>
+<wire x1="2.15326875" y1="18.5166" x2="1.4986" y2="17.86193125" width="0.2032" layer="1"/>
+<wire x1="1.4986" y1="17.86193125" x2="1.4986" y2="16.93606875" width="0.2032" layer="1"/>
+<wire x1="10.16" y1="17.78" x2="5.44133125" y2="17.78" width="0.2032" layer="1"/>
+<wire x1="5.44133125" y1="17.78" x2="4.70473125" y2="18.5166" width="0.2032" layer="1"/>
+<wire x1="1.4986" y1="16.93606875" x2="3.429" y2="15.00566875" width="0.2032" layer="1"/>
+<wire x1="3.429" y1="15.00566875" x2="3.429" y2="14.859" width="0.2032" layer="1"/>
+<wire x1="24.257" y1="14.605" x2="24.257" y2="14.097" width="0.2032" layer="1"/>
+<wire x1="18.63170625" y1="10.16" x2="17.78" y2="10.16" width="0.2032" layer="1"/>
+<wire x1="21.5138" y1="11.3538" x2="19.82550625" y2="11.3538" width="0.2032" layer="1"/>
+<wire x1="19.82550625" y1="11.3538" x2="18.63170625" y2="10.16" width="0.2032" layer="1"/>
+<wire x1="24.257" y1="14.097" x2="21.5138" y2="11.3538" width="0.2032" layer="1"/>
+<wire x1="21.844" y1="26.609" x2="24.13" y2="26.609" width="0.2032" layer="1"/>
+<wire x1="24.13" y1="26.609" x2="25.4" y2="26.609" width="0.2032" layer="1"/>
+<wire x1="25.4" y1="26.609" x2="37.46" y2="26.609" width="0.2032" layer="1"/>
+<wire x1="37.46" y1="26.609" x2="38.227" y2="25.842" width="0.2032" layer="1"/>
+<wire x1="17.526" y1="26.559" x2="14.3985" y2="23.4315" width="0.2032" layer="1"/>
+<wire x1="14.3985" y1="23.4315" x2="12.00225" y2="23.4315" width="0.2032" layer="1"/>
+<wire x1="11.32025" y1="22.7495" x2="8.7795" y2="22.7495" width="0.2032" layer="1"/>
+<wire x1="12.00225" y1="23.4315" x2="11.32025" y2="22.7495" width="0.2032" layer="1"/>
+<via x="16.51" y="45.6906" extent="1-16" drill="0.508"/>
+<wire x1="16.51" y1="45.6906" x2="12.7294" y2="41.91" width="0.2032" layer="1"/>
+<wire x1="12.7294" y1="41.91" x2="12.7" y2="41.91" width="0.2032" layer="1"/>
+<via x="12.7" y="41.91" extent="1-16" drill="0.508"/>
+<wire x1="12.7" y1="41.91" x2="12.7" y2="40.64" width="0.2032" layer="16"/>
+<wire x1="12.7" y1="40.64" x2="12.7" y2="38.1" width="0.2032" layer="16"/>
+<wire x1="12.7" y1="38.1" x2="11.43" y2="36.83" width="0.2032" layer="16"/>
+<via x="11.43" y="36.83" extent="1-16" drill="0.508"/>
+<wire x1="11.43" y1="36.83" x2="14.031" y2="36.83" width="0.2032" layer="1"/>
+<wire x1="14.031" y1="36.83" x2="14.224" y2="36.637" width="0.2032" layer="1"/>
+<wire x1="16.51" y1="49.53" x2="16.51" y2="45.6906" width="0.2032" layer="16"/>
+<wire x1="12.7" y1="40.64" x2="15.6336" y2="40.64" width="0.2032" layer="16"/>
+<wire x1="15.6336" y1="40.64" x2="18.1736" y2="38.1" width="0.2032" layer="16"/>
+<via x="18.1736" y="38.1" extent="1-16" drill="0.508"/>
+<wire x1="18.1736" y1="38.1" x2="18.2346" y2="38.161" width="0.2032" layer="1"/>
+<wire x1="18.2346" y1="38.161" x2="20.066" y2="38.161" width="0.2032" layer="1"/>
+<wire x1="2.921" y1="34.163" x2="0" y2="31.242" width="0.2032" layer="16"/>
+<wire x1="0" y1="31.242" x2="0" y2="15.24" width="0.2032" layer="16"/>
+<wire x1="0" y1="15.24" x2="0.381" y2="14.859" width="0.2032" layer="16"/>
+<wire x1="0.381" y1="14.859" x2="3.429" y2="14.859" width="0.2032" layer="16"/>
+<wire x1="18.693" y1="32.127" x2="18.7482" y2="32.0718" width="0.2032" layer="1"/>
+<wire x1="18.7482" y1="32.0718" x2="19.21925" y2="32.0718" width="0.2032" layer="1"/>
+<wire x1="19.41405" y1="31.877" x2="20.193" y2="31.877" width="0.2032" layer="1"/>
+<wire x1="19.21925" y1="32.0718" x2="19.41405" y2="31.877" width="0.2032" layer="1"/>
+<wire x1="25.4" y1="26.609" x2="18.693" y2="32.127" width="0" layer="19" extent="1-1"/>
+<wire x1="14.224" y1="36.637" x2="21.693" y2="32.627" width="0" layer="19" extent="1-1"/>
+<wire x1="24.13" y1="26.609" x2="24.13" y2="26.609" width="0.2032" layer="1"/>
 </signal>
 <signal name="VCC">
@@
 <contactref element="R7" pad="1"/>
 <contactref element="X4" pad="9"/>
-<wire x1="22.225" y1="37.404" x2="22.225" y2="34.659" width="0.2032" layer="1"/>
-<wire x1="22.225" y1="34.659" x2="20.943" y2="33.377" width="0.2032" layer="1"/>
+<wire x1="22.225" y1="37.404" x2="22.225" y2="35.929" width="0.2032" layer="1"/>
+<wire x1="22.225" y1="35.929" x2="21.723" y2="35.427" width="0.2032" layer="1"/>
+<wire x1="21.723" y1="35.427" x2="21.723" y2="34.157" width="0.2032" layer="1"/>
+<wire x1="21.723" y1="34.157" x2="20.943" y2="33.377" width="0.2032" layer="1"/>
 </signal>
 <signal name="ISET">
@@
 <wire x1="18.681" y1="32.627" x2="17.272" y2="34.036" width="0.2032" layer="1"/>
 <wire x1="13.208" y1="26.3017" x2="13.208" y2="28.956" width="0.2032" layer="1"/>
-<wire x1="12.573" y1="29.591" x2="12.573" y2="32.639" width="0.2032" layer="1"/>
 <via x="12.573" y="32.639" extent="1-16" drill="0.508"/>
-<wire x1="13.208" y1="28.956" x2="12.573" y2="29.591" width="0.2032" layer="1"/>
+<wire x1="13.208" y1="28.956" x2="12.827" y2="29.337" width="0.2032" layer="1"/>
+<wire x1="12.827" y1="29.337" x2="12.573" y2="29.591" width="0.2032" layer="1"/>
+<wire x1="12.573" y1="29.591" x2="11.43" y2="30.734" width="0.2032" layer="1"/>
+<wire x1="11.43" y1="30.734" x2="11.43" y2="31.75" width="0.2032" layer="1"/>
+<wire x1="11.43" y1="31.75" x2="12.319" y2="32.639" width="0.2032" layer="1"/>
+<wire x1="12.319" y1="32.639" x2="12.573" y2="32.639" width="0.2032" layer="1"/>
 </signal>
 <signal name="CHARGER_IN">

Commit message: All air wires good
Parts:
- moved R11 1.80 mm to (25.0, 30.5)
Routing:
- net GND: track 228.4 -> 246.6 mm, vias 7 -> 9
- net VBAT: track 43.3 -> 48.1 mm
- net !PGOOD: track 2.61 -> 4.40 mm
- net N$4: track 23.9 -> 25.2 mm
Changed lines of the file:
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@@
 <drawing>
 <settings>
-<setting alwaysvectorfont="no"/>
+<setting alwaysvectorfont="yes"/>
 <setting verticaltext="up"/>
 </settings>
@@
 <element name="R4" library="adafruit" library_urn="urn:adsk.eagle:library:420" package="M0805" package3d_urn="urn:adsk.eagle:package:6240587/1" value="1K" x="16.256" y="37.211" smashed="yes" rot="R90"/>
 <element name="C5" library="adafruit" library_urn="urn:adsk.eagle:library:420" package="C0805K" package3d_urn="urn:adsk.eagle:package:6240397/1" value="10uF" x="19.685" y="27.559" smashed="yes" rot="R270"/>
-<element name="R11" library="adafruit" library_urn="urn:adsk.eagle:library:420" package="M0805" package3d_urn="urn:adsk.eagle:package:6240587/1" value="1K" x="23.749" y="31.75" smashed="yes" rot="R90"/>
+<element name="R11" library="adafruit" library_urn="urn:adsk.eagle:library:420" package="M0805" package3d_urn="urn:adsk.eagle:package:6240587/1" value="1K" x="25.019" y="30.48" smashed="yes" rot="R90"/>
 <element name="R8" library="adafruit" library_urn="urn:adsk.eagle:library:420" package="M0805" package3d_urn="urn:adsk.eagle:package:6240587/1" value="10K" x="21.844" y="27.559" smashed="yes" rot="R270"/>
 <element name="JP8" library="pinhead" library_urn="urn:adsk.eagle:library:325" package="1X02" package3d_urn="urn:adsk.eagle:package:22435/2" value="" x="2.921" y="35.433" smashed="yes" rot="R270">
@@
 <wire x1="19.82550625" y1="11.3538" x2="18.63170625" y2="10.16" width="0.2032" layer="1"/>
 <wire x1="24.257" y1="14.097" x2="21.5138" y2="11.3538" width="0.2032" layer="1"/>
-<wire x1="21.844" y1="26.609" x2="24.13" y2="26.609" width="0.2032" layer="1"/>
-<wire x1="24.13" y1="26.609" x2="25.4" y2="26.609" width="0.2032" layer="1"/>
-<wire x1="25.4" y1="26.609" x2="37.46" y2="26.609" width="0.2032" layer="1"/>
+<wire x1="21.844" y1="26.609" x2="37.46" y2="26.609" width="0.2032" layer="1"/>
 <wire x1="37.46" y1="26.609" x2="38.227" y2="25.842" width="0.2032" layer="1"/>
 <wire x1="17.526" y1="26.559" x2="14.3985" y2="23.4315" width="0.2032" layer="1"/>
@@
 <wire x1="19.41405" y1="31.877" x2="20.193" y2="31.877" width="0.2032" layer="1"/>
 <wire x1="19.21925" y1="32.0718" x2="19.41405" y2="31.877" width="0.2032" layer="1"/>
-<wire x1="25.4" y1="26.609" x2="18.693" y2="32.127" width="0" layer="19" extent="1-1"/>
-<wire x1="14.224" y1="36.637" x2="21.693" y2="32.627" width="0" layer="19" extent="1-1"/>
-<wire x1="24.13" y1="26.609" x2="24.13" y2="26.609" width="0.2032" layer="1"/>
+<wire x1="21.693" y1="31.627" x2="21.7482" y2="31.5718" width="0.2032" layer="1"/>
+<wire x1="21.7482" y1="31.5718" x2="22.21925" y2="31.5718" width="0.2032" layer="1"/>
+<wire x1="24.13" y1="28.53795" x2="24.13" y2="27.94" width="0.2032" layer="1"/>
+<wire x1="23.9142" y1="28.75375" x2="24.13" y2="28.53795" width="0.2032" layer="1"/>
+<wire x1="22.21925" y1="31.5718" x2="23.9142" y2="29.87685" width="0.2032" layer="1"/>
+<wire x1="23.9142" y1="29.87685" x2="23.9142" y2="28.75375" width="0.2032" layer="1"/>
+<wire x1="24.13" y1="27.94" x2="22.799" y2="26.609" width="0.2032" layer="1"/>
+<wire x1="22.799" y1="26.609" x2="21.844" y2="26.609" width="0.2032" layer="1"/>
+<wire x1="21.693" y1="32.627" x2="22.086" y2="33.02" width="0.2032" layer="1"/>
+<wire x1="22.086" y1="33.02" x2="22.86" y2="33.02" width="0.2032" layer="1"/>
+<wire x1="22.86" y1="33.02" x2="22.86" y2="33.458525" width="0.2032" layer="1"/>
+<wire x1="22.86" y1="33.458525" x2="22.517" y2="33.801525" width="0.2032" layer="1"/>
+<via x="22.517" y="33.801525" extent="1-16" drill="0.508"/>
+<wire x1="22.517" y1="33.801525" x2="19.538475" y2="33.801525" width="0.2032" layer="16"/>
+<wire x1="19.538475" y1="33.801525" x2="19.05" y2="34.29" width="0.2032" layer="16"/>
+<wire x1="19.05" y1="34.29" x2="18.6302" y2="34.29" width="0.2032" layer="16"/>
+<via x="18.6302" y="34.29" extent="1-16" drill="0.508"/>
+<wire x1="18.6302" y1="34.29" x2="18.6302" y2="37.6434" width="0.2032" layer="1"/>
+<wire x1="18.6302" y1="37.6434" x2="18.1736" y2="38.1" width="0.2032" layer="1"/>
 </signal>
 <signal name="VCC">
@@
 <contactref element="X4" pad="10"/>
 <contactref element="X4" pad="11"/>
-<wire x1="26.797" y1="34.925" x2="26.67" y2="34.925" width="0.2032" layer="1"/>
-<via x="23.495" y="34.925" extent="1-16" drill="0.508"/>
-<wire x1="26.67" y1="34.925" x2="23.495" y2="34.925" width="0.2032" layer="1"/>
-<wire x1="23.495" y1="34.925" x2="23.4698" y2="34.8998" width="0.2032" layer="16"/>
-<wire x1="23.4698" y1="34.8998" x2="20.955" y2="34.8998" width="0.2032" layer="16"/>
+<wire x1="22.86" y1="34.8998" x2="20.955" y2="34.8998" width="0.2032" layer="16"/>
 <wire x1="20.955" y1="34.8998" x2="20.701" y2="34.6458" width="0.2032" layer="16"/>
 <via x="20.701" y="34.6458" extent="1-16" drill="0.508"/>
@@
 <wire x1="5.08" y1="38.1" x2="5.3" y2="38.32" width="0.2032" layer="1"/>
 <wire x1="5.3" y1="38.32" x2="7.62" y2="38.32" width="0.2032" layer="1"/>
-<wire x1="22.6442" y1="30.02375" x2="22.82275" y2="29.8452" width="0.2032" layer="1"/>
-<wire x1="22.82275" y1="29.8452" x2="24.67525" y2="29.8452" width="0.2032" layer="1"/>
-<wire x1="24.67525" y1="29.8452" x2="24.8538" y2="30.02375" width="0.2032" layer="1"/>
-<wire x1="24.8538" y1="33.1088" x2="26.67" y2="34.925" width="0.2032" layer="1"/>
-<wire x1="21.693" y1="31.127" x2="22.6442" y2="30.1758" width="0.2032" layer="1"/>
-<wire x1="22.6442" y1="30.1758" x2="22.6442" y2="30.02375" width="0.2032" layer="1"/>
-<wire x1="24.8538" y1="30.02375" x2="24.8538" y2="33.1088" width="0.2032" layer="1"/>
+<wire x1="21.693" y1="31.127" x2="22.771375" y2="30.048625" width="0.2032" layer="1"/>
+<wire x1="22.771375" y1="30.048625" x2="22.771375" y2="29.8702" width="0.2032" layer="1"/>
+<via x="22.771375" y="29.8702" extent="1-16" drill="0.508"/>
+<wire x1="22.771375" y1="29.8702" x2="24.701575" y2="27.94" width="0.2032" layer="16"/>
+<wire x1="24.701575" y1="27.94" x2="26.67" y2="27.94" width="0.2032" layer="16"/>
+<wire x1="26.67" y1="27.94" x2="27.94" y2="29.21" width="0.2032" layer="16"/>
+<wire x1="27.94" y1="29.21" x2="27.94" y2="33.782" width="0.2032" layer="16"/>
+<wire x1="27.94" y1="33.782" x2="26.797" y2="34.925" width="0.2032" layer="16"/>
+<wire x1="26.7718" y1="34.8998" x2="26.797" y2="34.925" width="0.2032" layer="16"/>
+<wire x1="22.86" y1="34.8998" x2="26.7718" y2="34.8998" width="0.2032" layer="16"/>
 </signal>
 <signal name="A1">
@@
 <contactref element="X4" pad="7"/>
 <contactref element="R11" pad="1"/>
-<wire x1="23.749" y1="30.8" x2="22.422" y2="32.127" width="0.2032" layer="1"/>
+<wire x1="25.019" y1="29.53" x2="22.422" y2="32.127" width="0.2032" layer="1"/>
 <wire x1="22.422" y1="32.127" x2="21.693" y2="32.127" width="0.2032" layer="1"/>
 </signal>
@@
 <contactref element="R11" pad="2"/>
 <contactref element="PGOOD" pad="C"/>
-<wire x1="23.3298" y1="40.08025" x2="23.3298" y2="36.62775" width="0.2032" layer="1"/>
-<wire x1="23.3298" y1="36.62775" x2="22.6822" y2="35.98015" width="0.2032" layer="1"/>
-<wire x1="22.6822" y1="35.98015" x2="22.6822" y2="33.7668" width="0.2032" layer="1"/>
-<wire x1="22.6822" y1="33.7668" x2="23.749" y2="32.7" width="0.2032" layer="1"/>
+<wire x1="23.3298" y1="40.08025" x2="23.3298" y2="33.1192" width="0.2032" layer="1"/>
+<wire x1="23.3298" y1="33.1192" x2="25.019" y2="31.43" width="0.2032" layer="1"/>
 <wire x1="7.62" y1="40.42" x2="22.99005" y2="40.42" width="0.2032" layer="1"/>
 <wire x1="22.99005" y1="40.42" x2="23.3298" y2="40.08025" width="0.2032" layer="1"/>

Commit message: Final touches
Routing:
- net N$3: track 10.4 -> 9.57 mm
Other:
- board text added: "Woo & Burgos"
- board text removed: "Winnie Woo"
Changed lines of the file:
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@@
 <dimension x1="10.16" y1="-60.96" x2="10.414" y2="-63.5" x3="32.258" y3="-62.23" textsize="1.778" layer="47" dtype="vertical" unit="inch"/>
 <dimension x1="10.16" y1="-60.96" x2="29.21" y2="-58.547" x3="19.685" y3="-66.421" textsize="1.778" layer="47" dtype="horizontal" unit="inch"/>
-<text x="48.006" y="0.889" size="1.27" layer="21" ratio="12">Winnie Woo</text>
+<text x="45.466" y="0.889" size="1.27" layer="21" ratio="12">Woo &amp; Burgos</text>
 <text x="55.88" y="13.081" size="1.27" layer="21" font="vector" ratio="12" rot="R180">Hypnos1</text>
 <text x="56.134" y="37.973" size="1.27" layer="21" font="vector" ratio="12" rot="R180">Hypnos2</text>
@@
 <signal name="N$3">
 <contactref element="U1" pad="CSB"/>
-<wire x1="49.149" y1="26.162" x2="47.117" y2="26.162" width="0.2032" layer="1"/>
-<wire x1="47.117" y1="26.162" x2="46.482" y2="25.527" width="0.2032" layer="1"/>
-<wire x1="46.482" y1="25.527" x2="42.672" y2="25.527" width="0.2032" layer="1"/>
-<wire x1="42.149" y1="27.312" x2="42.149" y2="26.05" width="0.2032" layer="1"/>
-<wire x1="42.149" y1="26.05" x2="42.672" y2="25.527" width="0.2032" layer="1"/>
 <contactref element="SJ1" pad="2"/>
-<wire x1="49.149" y1="24.511" x2="49.149" y2="26.162" width="0.2032" layer="1"/>
+<wire x1="49.149" y1="24.511" x2="49.149" y2="25.781" width="0.2032" layer="1"/>
+<wire x1="49.149" y1="25.781" x2="48.26" y2="26.67" width="0.2032" layer="1"/>
+<wire x1="42.87275" y1="26.1622" x2="42.6942" y2="26.34075" width="0.2032" layer="1"/>
+<wire x1="42.6942" y1="26.34075" x2="42.6942" y2="26.7668" width="0.2032" layer="1"/>
+<wire x1="42.6942" y1="26.7668" x2="42.149" y2="27.312" width="0.2032" layer="1"/>
+<wire x1="45.27525" y1="26.1622" x2="42.87275" y2="26.1622" width="0.2032" layer="1"/>
+<wire x1="48.26" y1="26.67" x2="45.78305" y2="26.67" width="0.2032" layer="1"/>
+<wire x1="45.78305" y1="26.67" x2="45.27525" y2="26.1622" width="0.2032" layer="1"/>
 </signal>
 <signal name="VLIPO">
