File: PCB/Adaptor Board/WC Adaptor.sch (EAGLE design)
At the start: 5 parts, among them J1 1725672

Commit message: Add files via upload
Changed lines of the file:
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@@
 <instance part="J1" gate="G$1" x="66.04" y="97.79" smashed="yes" rot="R180">
 <attribute name="NAME" x="49.53" y="90.17" size="1.778" layer="95" rot="R180" align="center-left"/>
-<attribute name="VALUE" x="49.53" y="92.71" size="1.778" layer="96" rot="R180" align="center-left"/>
+<attribute name="VALUE" x="57.15" y="92.71" size="1.778" layer="96" rot="R180" align="center-left"/>
 </instance>
 </instances>
