File: PCB/v2.7/Chime PCB v2.7_9.18.brd (EAGLE design)
At the start: 64.8 x 78.8 mm, 31 parts, among them J1_SPI 1725698, J2_I2C 1725672, J4_A1 282834-3, J5_A0 282834-3, U1 MS5803-02BA, X4 BQ24074

Commit message: Adding final I2C_Extender and Chime PCB board file
Parts:
- removed J4_A1: 282834-3, Fixed Terminal Blocks 3P:TE_282834-3
- added C3: 15nF, rcl:C0805
- added CHG: (no value), adafruit:CHIPLED_0805
- added J2_I2C1: 1725672, 1725672:1725672
- added PGOOD: PGOOD, adafruit:CHIPLED_0805
- added R5, R6: 22K, adafruit:M0805
- moved J1_SPI 16.6 mm to (44.5, 49.5)
- moved J2_I2C 16.6 mm to (29.2, 49.5)
- moved J5_A0 16.6 mm to (3.81, 49.5)
- moved U$3 12.7 mm to (3.81, 62.2)
- moved U$4 12.7 mm to (58.5, 62.1)
- moved R11 1.80 mm to (25.0, 30.5)
- moved R3 1.27 mm to (18.8, 37.2)
Connections:
- removed net N$1: X4.5
- new net N$4: PGOOD.C, R11.2
- new net N$5: CHG.C, R7.2
- new net SIGNAL: J5_A0.2, R5.2, R6.1
- net A0: now also C3.1, R5.1; no longer J5_A0.2
- net A1: now also J1_SPI.3; no longer J4_A1.2
- net A3: no longer J1_SPI.3
- net GND: now also C3.2, J2_I2C1.2, JP9.2, R6.2; no longer J4_A1.1
- net SCL: now also J2_I2C1.3
- net SDA: now also J2_I2C1.4
- net VBAT: now also CHG.A, PGOOD.A, X4.5
- net VCC: now also J2_I2C1.1; no longer J4_A1.3
Routing:
- net VCC: track 161.6 -> 19.4 mm, vias 0 -> 1
- net SIGNAL: track 0.00 -> 75.9 mm
- net A3: track 63.8 -> 0.00 mm
- net N$4: track 0.00 -> 54.7 mm, vias 0 -> 2
- net A0: track 60.1 -> 14.8 mm
- net VBAT: track 8.09 -> 48.1 mm, vias 2 -> 3
- net N$5: track 0.00 -> 32.0 mm
- net MOSI: track 63.7 -> 42.4 mm, vias 0 -> 1
- net A1: track 60.3 -> 81.5 mm
- net GND: track 19.8 -> 40.4 mm
- net SCK: track 65.5 -> 44.9 mm
- net SCL: track 49.8 -> 67.0 mm
- net !PGOOD: track 2.61 -> 10.9 mm, vias 0 -> 2
- net MISO: track 62.8 -> 54.6 mm
- net 5VRAIL: track 26.3 -> 34.1 mm
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Other:
- board size 64.8 x 78.8 mm -> 64.8 x 68.6 mm
- board text added: "+"
- board text added: "-"
- board text added: ".015uF"
- board text added: "10K"
- board text added: "10uF"
- board text added: "1K"
- board text added: "22K"
- board text added: "Chime v2.7 9.18.23"
- board text added: "SIGNAL"
- board text added: "Woo & Burgos"
- board text removed: "A0"
- board text removed: "A3"
- board text removed: "Chime v2.1"
- board text removed: "Winnie Woo"
